Commit message: depth camera functional

File: open_project/urdf/tello_seeker.urdf (robot description, URDF)
Before this commit: robot tello_seeker, 3 links, 2 joints
Links:
- removed link downward_depth_camera_link
- added link depth_camera_link, mass 0.1; visual box size=0.05 0.05 0.05
Joints:
- removed joint downward_depth_camera_joint
- added joint depth_camera_joint: type fixed, parent base_link, child depth_camera_link, origin xyz=0 0 -0.1 rpy=0 1.5708 0

Commit message: edit stuff

File: open_project/urdf/tello_seeker.urdf (robot description, URDF)
Before this commit: robot tello_seeker, 3 links, 2 joints
Links:
- removed link base_link
- added link robot1/base_link, mass 0.1; collision box size=0.18 0.18 0.05; visual box size=0.07 0.02 0.02
Joints:
- joint camera_joint: parent base_link -> robot1/base_link
- joint depth_camera_joint: parent base_link -> robot1/base_link
